Commit message: debugged previous upload; simulation runs now with roslaunch

File: mani_description/urdf/mani.urdf.xacro (robot description, xacro)
@@ -15,5 +15,5 @@
 			<origin xyz="0 0 0" rpy="${PI} 0 0"/>
 			<geometry>
-				<mesh filename="file://$(find mani)/mani_description/meshes/MANI-chassis.STL" scale="${to_scale} ${to_scale} ${to_scale}"/>
+				<mesh filename="file://$(find manisim)/mani_description/meshes/MANI-chassis.STL" scale="${to_scale} ${to_scale} ${to_scale}"/>
 			</geometry>
 		</visual>
@@ -21,5 +21,5 @@
                 	<origin xyz="0 0 0" rpy="${PI} 0 0"/>
 			<geometry>
-				<mesh filename="file://$(find mani)/mani_description/meshes/MANI-chassis.STL" scale="${to_scale} ${to_scale} ${to_scale}"/>
+				<mesh filename="file://$(find manisim)/mani_description/meshes/MANI-chassis.STL" scale="${to_scale} ${to_scale} ${to_scale}"/>
 			</geometry>
 		</collision>
@@ -43,5 +43,5 @@
 			<origin xyz="0 0 0"/>
 			<geometry>
-				<mesh filename="file://$(find mani)/mani_description/meshes/MANI-cameraneck.STL" scale="${to_scale} ${to_scale} ${to_scale}"/>
+				<mesh filename="file://$(find manisim)/mani_description/meshes/MANI-cameraneck.STL" scale="${to_scale} ${to_scale} ${to_scale}"/>
 			</geometry>
 		</visual>
@@ -49,5 +49,5 @@
 			<origin xyz="0 0 0"/>
                         <geometry>
-                               	<mesh filename="file://$(find mani)/mani_description/meshes/MANI-cameraneck.STL" scale="${to_scale} ${to_scale} ${to_scale}"/>
+                               	<mesh filename="file://$(find manisim)/mani_description/meshes/MANI-cameraneck.STL" scale="${to_scale} ${to_scale} ${to_scale}"/>
                         </geometry>
 		</collision>
@@ -71,5 +71,5 @@
 			<origin xyz="0 0 0"/>
 			<geometry>
-				<mesh filename="file://$(find mani)/mani_description/meshes/MANI-camerahead.STL" scale="${to_scale} ${to_scale} ${to_scale}"/>
+				<mesh filename="file://$(find manisim)/mani_description/meshes/MANI-camerahead.STL" scale="${to_scale} ${to_scale} ${to_scale}"/>
 			</geometry>
 		</visual>
@@ -77,5 +77,5 @@
 			<origin xyz="0 0 0"/>
 			<geometry>
-				<mesh filename="file://$(find mani)/mani_description/meshes/MANI-camerahead.STL" scale="${to_scale} ${to_scale} ${to_scale}"/>
+				<mesh filename="file://$(find manisim)/mani_description/meshes/MANI-camerahead.STL" scale="${to_scale} ${to_scale} ${to_scale}"/>
 			</geometry>
 		</collision>
@@ -129,5 +129,5 @@
                     		<xacro:insert_block name="visual_origin"/>
                         	<geometry>
-                                	<mesh filename="file://$(find mani)/mani_description/meshes/MANI-steeringangle.STL" scale="${to_scale} ${to_scale} ${to_scale}"/>
+                                	<mesh filename="file://$(find manisim)/mani_description/meshes/MANI-steeringangle.STL" scale="${to_scale} ${to_scale} ${to_scale}"/>
                         	</geometry>
                 	</visual>
@@ -135,5 +135,5 @@
                         	<xacro:insert_block name="collision_origin"/>
                         	<geometry>
-                            		<mesh filename="file://$(find mani)/mani_description/meshes/MANI-steeringangle.STL" scale="${to_scale} ${to_scale} ${to_scale}"/>
+                            		<mesh filename="file://$(find manisim)/mani_description/meshes/MANI-steeringangle.STL" scale="${to_scale} ${to_scale} ${to_scale}"/>
                              </geometry>
                 	</collision>
@@ -182,5 +182,5 @@
 				<xacro:insert_block name="visual_origin"/>
                         	<geometry>
-                                	<mesh filename="file://$(find mani)/mani_description/meshes/MANI-wheel.STL" scale="${to_scale} ${to_scale} ${to_scale}"/>
+                                	<mesh filename="file://$(find manisim)/mani_description/meshes/MANI-wheel.STL" scale="${to_scale} ${to_scale} ${to_scale}"/>
                         	</geometry>
                 	</visual>
