Commit message: renamed camera links/joints and changed license in package.xml

File: manisim_description/urdf/manisim.urdf.xacro (robot description, xacro)
@@ -229,5 +229,5 @@
         </wheel>
 	<!-- camera head 60-60 grad-->
-	<joint name="cam_1_neck" type="revolute"> <!-- revolute -->
+	<joint name="cam_pan" type="revolute"> <!-- revolute -->
 		<parent link="chassis"/>
 		<child link="camera_pan"/>
@@ -239,5 +239,5 @@
 	<xacro:property name="campan_dz" value="0.09846"/>
 	<xacro:property name="campan_dy" value="0.097975"/>
-	<joint name="cam_2_head" type="revolute">
+	<joint name="cam_tilt" type="revolute">
 		<parent link="camera_pan"/>
 		<child link="camera_tilt"/>
@@ -311,20 +311,20 @@
 	<!-- transmission -->
         <!-- move camera neck/head -->
-	<transmission name="transm_cam_neck">
+	<transmission name="transm_camera_pan">
 		<type>transmission_interface/SimpleTransmission</type>
-		<joint name="cam_1_neck">
+		<joint name="cam_pan">
 			<hardwareInterface>hardware_interface/EffortJointInterface</hardwareInterface>
 		</joint>
-		<actuator name="motor_cam_neck">
+		<actuator name="motor_camera_pan">
 			<hardwareInterface>EffortJointInterface</hardwareInterface>
 			<mechanicalReduction>1</mechanicalReduction>
 		</actuator>
 	</transmission>
-	<transmission name="transm_cam_head">
+	<transmission name="transm_camera_tilt">
 		<type>transmission_interface/SimpleTransmission</type>
-		<joint name="cam_2_head">
+		<joint name="cam_tilt">
 			<hardwareInterface>hardware_interface/EffortJointInterface</hardwareInterface>
 		</joint>
-		<actuator name="motor_cam_head">
+		<actuator name="motor_camera_tilt">
 			<hardwareInterface>EffortJointInterface</hardwareInterface>
 			<mechanicalReduction>1</mechanicalReduction>
